Commit message: Fixed near zero offsets in huboplus.urdf

File: huboplus.urdf (robot description, URDF)
Before this commit: robot huboplus, 58 links, 57 joints
Joints:
- joint LAR: origin xyz=0.0711787 -0.0466006 -1.04e-10 rpy=0 -0 0 -> xyz=0.0711787 -0.0466006 0 rpy=0 -0 0
- joint LHP: origin xyz=-0.0529074 0.0655748 9.99159e-05 rpy=0 -0 0 -> xyz=-0.052 0.0655748 0 rpy=0 -0 0
- joint LHR: origin xyz=0.0520001 1.50498e-06 -0.091004 rpy=0 -0 0 -> xyz=0.052 0 -0.091004 rpy=0 -0 0
- joint LSY: origin xyz=-0.0269 -0.000166249 -0.0245 rpy=0 -0 0 -> xyz=-0.0269 0 -0.0245 rpy=0 -0 0
- joint LWP: origin xyz=1.72973e-06 -0.00872953 -0.05255 rpy=0 -0 0 -> xyz=0 -0.00872953 -0.05255 rpy=0 -0 0
- joint RAR: origin xyz=0.0711787 0.0466006 -1.04e-10 rpy=0 -0 0 -> xyz=0.0711787 0.0466006 0 rpy=0 -0 0
- joint RHP: origin xyz=-0.0529074 -0.0655748 9.99159e-05 rpy=0 -0 0 -> xyz=-0.0520 -0.0655748 0 rpy=0 -0 0
- joint RHR: origin xyz=0.0520001 7.3455e-05 -0.091004 rpy=0 -0 0 -> xyz=0.052 0 -0.091004 rpy=0 -0 0
- joint RWP: origin xyz=1.72973e-06 0.01 -0.05255 rpy=0 -0 0 -> xyz=0 0.01 -0.05255 rpy=0 -0 0

File: hubosimple.urdf (robot description, URDF)
Before this commit: robot jaemiHubo, 66 links, 65 joints
Joints:
- joint LAR: origin xyz=0.071244 -0.0465 -1.6e-05 rpy=0 -0 0 -> xyz=0.071244 -0.0465 0 rpy=0 -0 0
- joint RAR: origin xyz=0.071244 0.0465 -1.6e-05 rpy=0 -0 0 -> xyz=0.071244 0.0465 0 rpy=0 -0 0

Commit message: Additional alignments made to knee pitch and wrist to make 2DOF joints coincide with 3DOF joints

File: huboplus.urdf (robot description, URDF)
Before this commit: robot huboplus, 58 links, 57 joints
Joints:
- joint LKP: origin xyz=0.000766364 -0.0445011 -0.280007 rpy=0 -0 0 -> xyz=0 -0.0445011 -0.280007 rpy=0 -0 0
- joint LWY: origin xyz=-0.0219906 0.018 -0.111408 rpy=0 -0 0 -> xyz=-0.0219936 0.018 -0.111408 rpy=0 -0 0
- joint RKP: origin xyz=0.000766364 0.0445011 -0.280007 rpy=0 -0 0 -> xyz=0 0.0445011 -0.280007 rpy=0 -0 0
- joint RWY: origin xyz=-0.0219906 -0.018 -0.111408 rpy=0 -0 0 -> xyz=-0.0219936 -0.018 -0.111408 rpy=0 -0 0
